Commit message: Updated xacro to be more minimal. Added config packages

File: description/picknik_ur5e.xacro (robot description, xacro)
@@ -4,6 +4,4 @@
   <xacro:arg name="use_fake_hardware" default="false" />
   <xacro:arg name="external_camera" default="false" />
-  <xacro:arg name="has_tool_changer" default="true" />
-  <xacro:arg name="use_pinch_link" default="true" />
   <xacro:arg name="name" default="" />
   <xacro:arg name="joint_limits_parameters_file" default="" />
@@ -11,23 +9,15 @@
   <xacro:arg name="physical_parameters_file" default="" />
   <xacro:arg name="visual_parameters_file" default="" />
-  <xacro:arg name="headless_mode" default="false" />
   <xacro:arg name="robot_ip" default="0.0.0.0" />
-  <xacro:if value="$(arg has_tool_changer)">
-    <xacro:property name="camera_adapter_parent" value="tool_changer_tool0" />
-  </xacro:if>
-  <xacro:unless value="$(arg has_tool_changer)">
-    <xacro:property name="camera_adapter_parent" value="tool0" />
-  </xacro:unless>
+  <xacro:property name="camera_adapter_parent" value="tool0" />
   <!-- Import macros for main hardware components -->
   <xacro:include filename="$(find ur_description)/urdf/ur_macro.xacro" />
   <xacro:include filename="$(find robotiq_description)/urdf/ur_to_robotiq_adapter.urdf.xacro" />
   <xacro:include filename="$(find robotiq_description)/urdf/robotiq_gripper_macro.urdf.xacro" />
-  <xacro:include filename="$(find picknik_accessories)/descriptions/brackets/mtc_ur_tool_changer/mtc_ur_tool_changer.urdf.xacro" />
   <xacro:include filename="$(find picknik_accessories)/descriptions/brackets/ur_realsense_camera_adapter/picknik_ur_camera_adapter.urdf.xacro" />
   <xacro:include filename="$(find picknik_accessories)/descriptions/sensors/realsense_d415.urdf.xacro" />
   <xacro:include filename="$(find picknik_accessories)/descriptions/sensors/realsense_d435.urdf.xacro" />
-  <xacro:include filename="$(find picknik_ur_base_config)/description/pinch_link.xacro" />
   <!-- Initial positions for simulations (Mock Hardware and Gazebo) -->
-  <xacro:arg name="initial_positions_file" default="$(find picknik_ur_base_config)/config/initial_positions.yaml"/>
+  <xacro:arg name="initial_positions_file" default="$(find ur_base_config)/config/initial_positions.yaml"/>
   <xacro:property name="initial_positions_file" default="$(arg initial_positions_file)"/>
   <!-- Import environment macros -->
@@ -46,5 +36,4 @@
     use_fake_hardware="$(arg use_fake_hardware)"
     initial_positions="${xacro.load_yaml(initial_positions_file)}"
-    headless_mode="$(arg headless_mode)"
     robot_ip="$(arg robot_ip)"
     script_filename="$(find ur_robot_driver)/resources/ros_control.urscript"
@@ -53,12 +42,4 @@
     <origin xyz="0 0 0" rpy="0 0 0" />
   </xacro:ur_robot>
-  <xacro:if value="$(arg has_tool_changer)">
-    <!-- tool changer-->
-    <xacro:mtc_ur_tool_changer prefix="" connected_to="tool0" rotation="0" />
-  </xacro:if>
-  <!-- pinch geometry for moveit motion planning. see https://github.com/UniversalRobots/Universal_Robots_ROS2_Driver/issues/611 -->
-  <xacro:if value="$(arg use_pinch_link)">
-    <xacro:pinch_link prefix="" />
-  </xacro:if>
   <!-- wrist camera adapter and camera-->
   <xacro:ur_realsense_camera_adapter prefix="" connected_to="${camera_adapter_parent}" rotation="0" />
