Commit message: Removed tool changer link from gripper camera xacro. Added initial urdf and srdf

File: description/gripper_and_camera.xacro (robot description, xacro)
@@ -15,12 +15,6 @@
     <origin xyz="0.0 -0.016124 -0.18430" rpy="${pi / 180.0 * 5} 0 -${pi}" />
   </joint>
-  <link name="tool_changer_tool0" />
-  <joint name="tool_side_joint" type="fixed">
-    <parent link="tool0" />
-    <child link="tool_changer_tool0" />
-    <origin xyz="0 0 0.0331" rpy="0 0 0" />
-  </joint>
   <!-- wrist camera adapter and camera-->
-  <xacro:ur_realsense_camera_adapter prefix="" connected_to="tool_changer_tool0" rotation="0"/>
+  <xacro:ur_realsense_camera_adapter prefix="" connected_to="tool0" rotation="0"/>
   <xacro:realsense_d415 parent="d415_mount_link" name="wrist_mounted_camera">
     <origin xyz="0 0 0" rpy="0 0 0"/>
