Commit message: Removed boxes from urdf environment for now

File: src/ur_base_config/description/robot.urdf (robot description, URDF)
Before this commit: robot ur5e, 57 links, 56 joints
Links:
- removed link box_1
- removed link box_2
- removed link box_3
- removed link box_4
- removed link box_5
Joints:
- removed joint box1_on_table
- removed joint box2_on_table
- removed joint box3_on_table
- removed joint box4_on_table
- removed joint box5_on_table

File: starter_files/description/ur5e.xacro (robot description, xacro)
@@ -86,59 +86,4 @@
     <origin rpy="0 0 0" xyz="0 0 -0.05" />
   </joint>
-  <link name="box_1">
-    <xacro:cube_visual length="0.05" width="0.05" height="0.05">
-      <origin xyz="0 0 0" rpy="0 0 0" />
-      <color rgba="0.1 0.1 0.1 0.9" />
-    </xacro:cube_visual>
-  </link>
-  <joint name="box1_on_table" type="fixed">
-    <parent link="environment" />
-    <child link="box_1" />
-    <origin rpy="0 0 0" xyz="0.65 -0.35 0.1" />
-  </joint>
-  <link name="box_2">
-    <xacro:cube_visual length="0.05" width="0.05" height="0.05">
-      <origin xyz="0 0 0" rpy="0 0 0" />
-      <color rgba="0.5 0.5 0.5 0.9" />
-    </xacro:cube_visual>
-  </link>
-  <joint name="box2_on_table" type="fixed">
-    <parent link="environment" />
-    <child link="box_2" />
-    <origin rpy="0 0 0" xyz="0.65 0.35 0.1" />
-  </joint>
-  <link name="box_3">
-    <xacro:cube_visual length="0.05" width="0.05" height="0.05">
-      <origin xyz="0 0 0" rpy="0 0 0" />
-      <color rgba="0.8 0.3 0.1 0.9" />
-    </xacro:cube_visual>
-  </link>
-  <joint name="box3_on_table" type="fixed">
-    <parent link="environment" />
-    <child link="box_3" />
-    <origin rpy="0 0 0" xyz="0.65 0 0.1" />
-  </joint>
-  <link name="box_4">
-    <xacro:cube_visual length="0.05" width="0.05" height="0.05">
-      <origin xyz="0 0 0" rpy="0 0 0" />
-      <color rgba="0.8 0.3 0.1 0.9" />
-    </xacro:cube_visual>
-  </link>
-  <joint name="box4_on_table" type="fixed">
-    <parent link="environment" />
-    <child link="box_4" />
-    <origin rpy="0 0 0" xyz="-0.65 0.25 0.1" />
-  </joint>
-  <link name="box_5">
-    <xacro:cube_visual length="0.05" width="0.05" height="0.05">
-      <origin xyz="0 0 0" rpy="0 0 0" />
-      <color rgba="0.1 0.3 0.8 0.9" />
-    </xacro:cube_visual>
-  </link>
-  <joint name="box5_on_table" type="fixed">
-    <parent link="environment" />
-    <child link="box_5" />
-    <origin rpy="0 0 0" xyz="-0.65 -0.25 0.1" />
-  </joint>
   <!-- External Camera -->
   <link name="external_camera_link" />
