Commit message: Start migrating to 4.0.0

File: src/ur_base_config/description/ur5e.xacro (robot description, xacro)
@@ -53,4 +53,5 @@
     <origin xyz="0 0 0" rpy="0 0 0" />
   </xacro:robotiq_gripper>
+  <!-- This link aligns the axes of the grasp frame to our required convention for motion planning tasks. -->
   <link name="grasp_link" />
   <joint name="grasp_link_joint" type="fixed">
@@ -58,11 +59,4 @@
     <child link="grasp_link" />
     <origin xyz="0.0 0.0 0.134" rpy="0.0 0.0 ${pi}" />
-  </joint>
-  <!-- Moveit Studio requires a link name called manual_grasp_link to perform quick tasks such as inspect surface -->
-  <link name="manual_grasp_link" />
-  <joint name="manual_grasp_joint" type="fixed">
-    <parent link="grasp_link" />
-    <child link="manual_grasp_link" />
-    <origin xyz="0 0 0" rpy="${pi / 180.0 * 5} 0 0" />
   </joint>
   <!-- Environment -->

Commit message: Remove ur_site_config package and polish up basic Objectives

File: src/ur_base_config/description/ur5e.xacro (robot description, xacro)
@@ -80,4 +80,37 @@
     <origin rpy="0 0 0" xyz="0 0 -0.05" />
   </joint>
+  <link name="box_red">
+    <xacro:cube_visual length="0.05" width="0.05" height="0.05">
+      <origin xyz="0 0 0" rpy="0 0 0" />
+      <color rgba="1.0 0.0 0.0 0.9" />
+    </xacro:cube_visual>
+  </link>
+  <joint name="box_red_on_table" type="fixed">
+    <parent link="environment" />
+    <child link="box_red" />
+    <origin rpy="0 0 0" xyz="0.65 -0.3 0.1" />
+  </joint>
+  <link name="box_green">
+    <xacro:cube_visual length="0.05" width="0.05" height="0.05">
+      <origin xyz="0 0 0" rpy="0 0 0" />
+      <color rgba="0.0 1.0 0.0 0.9" />
+    </xacro:cube_visual>
+  </link>
+  <joint name="box_green_on_table" type="fixed">
+    <parent link="environment" />
+    <child link="box_green" />
+    <origin rpy="0 0 0" xyz="0.65 0.3 0.1" />
+  </joint>
+  <link name="box_blue">
+    <xacro:cube_visual length="0.05" width="0.05" height="0.05">
+      <origin xyz="0 0 0" rpy="0 0 0" />
+      <color rgba="0.0 0.0 1.0 0.9" />
+    </xacro:cube_visual>
+  </link>
+  <joint name="box_blue_on_table" type="fixed">
+    <parent link="environment" />
+    <child link="box_blue" />
+    <origin rpy="0 0 0" xyz="0.65 0 0.1" />
+  </joint>
   <!-- External Camera -->
   <link name="external_camera_link" />

File: src/ur_gazebo_config/description/ur5e_gazebo.xacro (robot description, xacro)
@@ -52,4 +52,5 @@
     <origin xyz="0 0 0" rpy="0 0 0" />
   </xacro:robotiq_gripper>
+  <!-- This link aligns the axes of the grasp frame to our required convention for motion planning tasks. -->
   <link name="grasp_link" />
   <joint name="grasp_link_joint" type="fixed">
@@ -57,11 +58,4 @@
     <child link="grasp_link" />
     <origin xyz="0.0 0.0 0.134" rpy="0.0 0.0 ${pi}" />
-  </joint>
-  <!-- Moveit Studio requires a link name called manual_grasp_link to perform quick tasks such as inspect surface -->
-  <link name="manual_grasp_link" />
-  <joint name="manual_grasp_joint" type="fixed">
-    <parent link="grasp_link" />
-    <child link="manual_grasp_link" />
-    <origin xyz="0 0 0" rpy="${pi / 180.0 * 5} 0 0" />
   </joint>
   <!-- Environment -->

Commit message: Update config packages section and Gazebo config

File: src/ur_base_config/description/ur5e.xacro (robot description, xacro)
@@ -56,5 +56,5 @@
   <link name="grasp_link" />
   <joint name="grasp_link_joint" type="fixed">
-    <parent link="gripper_mount_link" />
+    <parent link="robotiq_85_base_link" />
     <child link="grasp_link" />
     <origin xyz="0.0 0.0 0.134" rpy="0.0 0.0 ${pi}" />

File: src/ur_gazebo_config/description/ur5e_gazebo.xacro (robot description, xacro)
@@ -55,5 +55,5 @@
   <link name="grasp_link" />
   <joint name="grasp_link_joint" type="fixed">
-    <parent link="gripper_mount_link" />
+    <parent link="robotiq_85_base_link" />
     <child link="grasp_link" />
     <origin xyz="0.0 0.0 0.134" rpy="0.0 0.0 ${pi}" />

File: src/ur_gazebo_config/description/ur5e_with_scene_camera_gazebo.xacro (robot description, xacro)
@@ -52,16 +52,10 @@
     <origin xyz="0 0 0" rpy="0 0 0" />
   </xacro:robotiq_gripper>
+  <!-- This link aligns the axes of the grasp frame to our required convention for motion planning tasks. -->
   <link name="grasp_link" />
   <joint name="grasp_link_joint" type="fixed">
-    <parent link="gripper_mount_link" />
+    <parent link="robotiq_85_base_link" />
     <child link="grasp_link" />
     <origin xyz="0.0 0.0 0.134" rpy="0.0 0.0 ${pi}" />
-  </joint>
-  <!-- Moveit Studio requires a link name called manual_grasp_link to perform quick tasks such as inspect surface -->
-  <link name="manual_grasp_link" />
-  <joint name="manual_grasp_joint" type="fixed">
-    <parent link="grasp_link" />
-    <child link="manual_grasp_link" />
-    <origin xyz="0 0 0" rpy="${pi / 180.0 * 5} 0 0" />
   </joint>
   <!-- Environment -->

File: src/ur_hardware_config/description/picknik_007_ur5e.xacro (robot description, xacro)
@@ -67,16 +67,10 @@
     <origin xyz="0 0 0" rpy="0 0 0" />
   </xacro:robotiq_gripper>
+  <!-- This link aligns the axes of the grasp frame to our required convention for motion planning tasks. -->
   <link name="grasp_link" />
   <joint name="grasp_link_joint" type="fixed">
-    <parent link="gripper_mount_link" />
+    <parent link="robotiq_85_base_link" />
     <child link="grasp_link" />
     <origin xyz="0.0 0.0 0.134" rpy="0.0 0.0 ${pi}" />
-  </joint>
-  <!-- Moveit Studio requires a link name called manual_grasp_link to perform quick tasks such as inspect surface -->
-  <link name="manual_grasp_link" />
-  <joint name="manual_grasp_joint" type="fixed">
-    <parent link="grasp_link" />
-    <child link="manual_grasp_link" />
-    <origin xyz="0 0 0" rpy="${pi / 180.0 * 5} 0 0" />
   </joint>
   <!-- Environment -->

File: starter_files/description/robot.urdf (robot description, URDF)
Before this commit: robot ur5e, 52 links, 51 joints
Links:
- removed link manual_grasp_link
Joints:
- removed joint manual_grasp_joint

Commit message: Update training materials to 4.0.0 (#23)

File: src/ur_base_config/description/ur5e.xacro (robot description, xacro)
@@ -53,16 +53,10 @@
     <origin xyz="0 0 0" rpy="0 0 0" />
   </xacro:robotiq_gripper>
+  <!-- This link aligns the axes of the grasp frame to our required convention for motion planning tasks. -->
   <link name="grasp_link" />
   <joint name="grasp_link_joint" type="fixed">
-    <parent link="gripper_mount_link" />
+    <parent link="robotiq_85_base_link" />
     <child link="grasp_link" />
     <origin xyz="0.0 0.0 0.134" rpy="0.0 0.0 ${pi}" />
-  </joint>
-  <!-- Moveit Studio requires a link name called manual_grasp_link to perform quick tasks such as inspect surface -->
-  <link name="manual_grasp_link" />
-  <joint name="manual_grasp_joint" type="fixed">
-    <parent link="grasp_link" />
-    <child link="manual_grasp_link" />
-    <origin xyz="0 0 0" rpy="${pi / 180.0 * 5} 0 0" />
   </joint>
   <!-- Environment -->
@@ -86,4 +80,37 @@
     <origin rpy="0 0 0" xyz="0 0 -0.05" />
   </joint>
+  <link name="box_red">
+    <xacro:cube_visual length="0.05" width="0.05" height="0.05">
+      <origin xyz="0 0 0" rpy="0 0 0" />
+      <color rgba="1.0 0.0 0.0 0.9" />
+    </xacro:cube_visual>
+  </link>
+  <joint name="box_red_on_table" type="fixed">
+    <parent link="environment" />
+    <child link="box_red" />
+    <origin rpy="0 0 0" xyz="0.65 -0.3 0.1" />
+  </joint>
+  <link name="box_green">
+    <xacro:cube_visual length="0.05" width="0.05" height="0.05">
+      <origin xyz="0 0 0" rpy="0 0 0" />
+      <color rgba="0.0 1.0 0.0 0.9" />
+    </xacro:cube_visual>
+  </link>
+  <joint name="box_green_on_table" type="fixed">
+    <parent link="environment" />
+    <child link="box_green" />
+    <origin rpy="0 0 0" xyz="0.65 0.3 0.1" />
+  </joint>
+  <link name="box_blue">
+    <xacro:cube_visual length="0.05" width="0.05" height="0.05">
+      <origin xyz="0 0 0" rpy="0 0 0" />
+      <color rgba="0.0 0.0 1.0 0.9" />
+    </xacro:cube_visual>
+  </link>
+  <joint name="box_blue_on_table" type="fixed">
+    <parent link="environment" />
+    <child link="box_blue" />
+    <origin rpy="0 0 0" xyz="0.65 0 0.1" />
+  </joint>
   <!-- External Camera -->
   <link name="external_camera_link" />

File: src/ur_gazebo_config/description/ur5e_gazebo.xacro (robot description, xacro)
@@ -52,16 +52,10 @@
     <origin xyz="0 0 0" rpy="0 0 0" />
   </xacro:robotiq_gripper>
+  <!-- This link aligns the axes of the grasp frame to our required convention for motion planning tasks. -->
   <link name="grasp_link" />
   <joint name="grasp_link_joint" type="fixed">
-    <parent link="gripper_mount_link" />
+    <parent link="robotiq_85_base_link" />
     <child link="grasp_link" />
     <origin xyz="0.0 0.0 0.134" rpy="0.0 0.0 ${pi}" />
-  </joint>
-  <!-- Moveit Studio requires a link name called manual_grasp_link to perform quick tasks such as inspect surface -->
-  <link name="manual_grasp_link" />
-  <joint name="manual_grasp_joint" type="fixed">
-    <parent link="grasp_link" />
-    <child link="manual_grasp_link" />
-    <origin xyz="0 0 0" rpy="${pi / 180.0 * 5} 0 0" />
   </joint>
   <!-- Environment -->

Commit message: Update ur_ws and fix description

File: src/ur_base_config/description/ur5e.xacro (robot description, xacro)
@@ -4,4 +4,5 @@
   <xacro:arg name="use_fake_hardware" default="false" />
   <xacro:arg name="external_camera" default="false" />
+  <xacro:arg name="has_tool_changer" default="true"/>
   <xacro:arg name="name" default="" />
   <xacro:arg name="joint_limits_parameters_file" default="" />
@@ -9,21 +10,26 @@
   <xacro:arg name="physical_parameters_file" default="" />
   <xacro:arg name="visual_parameters_file" default="" />
+  <xacro:arg name="headless_mode" default="false"/>
   <xacro:arg name="robot_ip" default="0.0.0.0" />
+  <xacro:arg name="use_tool_communication" default="false"/>
+  <xacro:arg name="tool_voltage" default="0"/>
+  <xacro:arg name="tool_device_name" default="/dev/ttyUSB0"/>
+  <xacro:arg name="simulation" default=""/>
   <xacro:property name="camera_adapter_parent" value="tool0" />
   <!-- Import macros for main hardware components -->
   <xacro:include filename="$(find ur_description)/urdf/ur_macro.xacro" />
-  <xacro:include filename="$(find robotiq_description)/urdf/ur_to_robotiq_adapter.urdf.xacro" />
-  <xacro:include filename="$(find robotiq_description)/urdf/robotiq_2f_85_macro.urdf.xacro" />
-  <xacro:include filename="$(find picknik_accessories)/descriptions/brackets/ur_realsense_camera_adapter/picknik_ur_camera_adapter.urdf.xacro" />
-  <xacro:include filename="$(find picknik_accessories)/descriptions/sensors/realsense_d415.urdf.xacro" />
-  <xacro:include filename="$(find picknik_accessories)/descriptions/sensors/realsense_d435.urdf.xacro" />
   <!-- Initial positions for simulations (Mock Hardware and Gazebo) -->
   <xacro:arg name="initial_positions_file" default="$(find ur_base_config)/config/initial_positions.yaml"/>
   <xacro:property name="initial_positions_file" default="$(arg initial_positions_file)"/>
-  <!-- Import environment macros -->
-  <xacro:include filename="$(find picknik_accessories)/descriptions/geometry/collision_and_visual/cube_collision_and_visual.urdf.xacro" />
-  <xacro:include filename="$(find picknik_accessories)/descriptions/geometry/visual/cube_visual.urdf.xacro" />
   <link name="world" />
   <!-- arm -->
+  <!-- Initial positions for simulations (Mock Hardware and Gazebo) -->
+  <xacro:property name="simulation" default="$(arg simulation)"/>
+  <xacro:if value="${simulation == 'gazebo'}">
+      <xacro:property name="use_fake_hardware" default="false"/>
+  </xacro:if>
+  <xacro:if value="${not simulation == 'gazebo'}">
+      <xacro:property name="use_fake_hardware" default="$(arg use_fake_hardware)"/>
+  </xacro:if>
   <xacro:ur_robot
     name="$(arg name)"
@@ -36,5 +42,10 @@
     use_fake_hardware="$(arg use_fake_hardware)"
     initial_positions="${xacro.load_yaml(initial_positions_file)}"
+    sim_ignition="${simulation == 'gazebo'}"
+    headless_mode="$(arg headless_mode)"
     robot_ip="$(arg robot_ip)"
+    use_tool_communication="$(arg use_tool_communication)"
+    tool_voltage="$(arg tool_voltage)"
+    tool_device_name="$(arg tool_device_name)"
     script_filename="$(find ur_robot_driver)/resources/ros_control.urscript"
     output_recipe_filename="$(find ur_robot_driver)/resources/rtde_output_recipe.txt"
@@ -42,84 +53,16 @@
     <origin xyz="0 0 0" rpy="0 0 0" />
   </xacro:ur_robot>
-  <!-- wrist camera adapter and camera-->
-  <xacro:ur_realsense_camera_adapter prefix="" connected_to="${camera_adapter_parent}" rotation="0" />
-  <xacro:realsense_d415 parent="d415_mount_link" name="wrist_mounted_camera">
-    <origin xyz="0 0 0" rpy="0 0 0" />
-  </xacro:realsense_d415>
-  <!-- Gripper and UR adapter-->
-  <xacro:ur_to_robotiq prefix="" connected_to="realsense_camera_adapter_tool0" rotation="0" />
-  <xacro:robotiq_gripper name="RobotiqGripperHardwareInterface" prefix=""
-    parent="gripper_mount_link" use_fake_hardware="$(arg use_fake_hardware)" com_port="/dev/ttyUSB0">
-    <origin xyz="0 0 0" rpy="0 0 0" />
-  </xacro:robotiq_gripper>
+  <!-- Gripper and UR adapter and realsense camera -->
+  <xacro:include filename="$(find ur_base_config)/description/ur_attachments_macro.xacro"/>
+  <xacro:ur_attachments parent="tool0" child="grasp_link" has_tool_changer="$(arg has_tool_changer)"/>
   <!-- This link aligns the axes of the grasp frame to our required convention for motion planning tasks. -->
   <link name="grasp_link" />
   <joint name="grasp_link_joint" type="fixed">
-    <parent link="robotiq_85_base_link" />
+    <parent link="tool0" />
     <child link="grasp_link" />
     <origin xyz="0.0 0.0 0.134" rpy="0.0 0.0 ${pi}" />
   </joint>
-  <!-- Environment -->
-  <link name="environment">
-    <visual>
-      <origin xyz="0 0 0" rpy="0 0 0" />
-      <geometry>
-        <mesh filename="package://picknik_accessories/descriptions/furniture/generic_table/wood_block.dae" scale="0.5 0.5 0.1"/>
-      </geometry>
-    </visual>
-    <collision>
-      <origin rpy="0 0 0" xyz="0 0 0"/>
-      <geometry>
-        <mesh filename="package://picknik_accessories/descriptions/furniture/generic_table/wood_block.dae" scale="0.5 0.5 0.1"/>
-      </geometry>
-    </collision>
-  </link>
-  <joint name="table_joint" type="fixed">
-    <parent link="base" />
-    <child link="environment" />
-    <origin rpy="0 0 0" xyz="0 0 -0.05" />
-  </joint>
-  <link name="box_red">
-    <xacro:cube_visual length="0.05" width="0.05" height="0.05">
-      <origin xyz="0 0 0" rpy="0 0 0" />
-      <color rgba="1.0 0.0 0.0 0.9" />
-    </xacro:cube_visual>
-  </link>
-  <joint name="box_red_on_table" type="fixed">
-    <parent link="environment" />
-    <child link="box_red" />
-    <origin rpy="0 0 0" xyz="0.65 -0.3 0.1" />
-  </joint>
-  <link name="box_green">
-    <xacro:cube_visual length="0.05" width="0.05" height="0.05">
-      <origin xyz="0 0 0" rpy="0 0 0" />
-      <color rgba="0.0 1.0 0.0 0.9" />
-    </xacro:cube_visual>
-  </link>
-  <joint name="box_green_on_table" type="fixed">
-    <parent link="environment" />
-    <child link="box_green" />
-    <origin rpy="0 0 0" xyz="0.65 0.3 0.1" />
-  </joint>
-  <link name="box_blue">
-    <xacro:cube_visual length="0.05" width="0.05" height="0.05">
-      <origin xyz="0 0 0" rpy="0 0 0" />
-      <color rgba="0.0 0.0 1.0 0.9" />
-    </xacro:cube_visual>
-  </link>
-  <joint name="box_blue_on_table" type="fixed">
-    <parent link="environment" />
-    <child link="box_blue" />
-    <origin rpy="0 0 0" xyz="0.65 0 0.1" />
-  </joint>
-  <!-- External Camera -->
-  <link name="external_camera_link" />
-  <joint name="external_camera_joint" type="fixed">
-    <parent link="world" />
-    <child link="external_camera_link" />
-    <origin xyz="-0.3 0.3 1.0" rpy="0.0 0.4 0" />
-  </joint>
-  <xacro:realsense_d435 parent="external_camera_link" name="scene_camera" visible="false">
-    <origin xyz="0 0 0" rpy="0 0 0" />
-  </xacro:realsense_d435>
+  <!-- Environment: contains scene geometry and external sensors, e.g. cameras -->
+  <xacro:include filename="$(find ur_base_config)/description/environment.xacro"/>
+  <xacro:environment parent="world"/>
 </robot>
