Commit message: Removed portions we will add in tutorials

File: src/ur_gazebo_config/description/ur5e_gazebo.xacro (robot description, xacro)
@@ -86,19 +86,4 @@
     <origin xyz="0.3 -0.3 1.0" rpy="0.0 0.4 3.14" />
   </joint>
-  <xacro:realsense_d435 parent="external_camera_link" name="scene_camera" visible="false" simulate_depth="true">
-    <origin xyz="0 0 0" rpy="0 0 0" />
-  </xacro:realsense_d435>
-  <!-- Additional Camera -->
-  <xacro:if value="$(arg use_extra_camera)">
-    <link name="extra_scene_camera_link" />
-    <joint name="extra_scene_camera_joint" type="fixed">
-      <parent link="world" />
-      <child link="extra_scene_camera_link" />
-      <origin xyz="-0.3 0.3 0.5" rpy="0.0 0.0 -3.14" />
-    </joint>
-    <xacro:realsense_d435 parent="extra_scene_camera_link" name="extra_camera" visible="false" simulate_depth="false">
-      <origin xyz="0 0 0" rpy="0 0 0" />
-    </xacro:realsense_d435>
-  </xacro:if>
   <!-- Force/Torque Sensor -->
   <link name="robot/wrist_3_joint/force_torque_sensor" />
