Commit message: Add Gazebo config modification solution files (#13)

File: src/ur_gazebo_config/description/ur5e_with_scene_camera_gazebo.xacro (robot description, xacro)
@@ -85,4 +85,17 @@
     <origin xyz="0.3 -0.3 1.0" rpy="0.0 0.4 3.14" />
   </joint>
+  <xacro:realsense_d435 parent="external_camera_link" name="scene_camera" visible="false" simulate_depth="true">
+    <origin xyz="0 0 0" rpy="0 0 0" />
+  </xacro:realsense_d435>
+  <!-- Additional Camera -->
+  <link name="extra_scene_camera_link" />
+  <joint name="extra_scene_camera_joint" type="fixed">
+    <parent link="world" />
+    <child link="extra_scene_camera_link" />
+    <origin xyz="-0.3 0.3 0.5" rpy="0.0 0.0 -3.14" />
+  </joint>
+  <xacro:realsense_d435 parent="extra_scene_camera_link" name="extra_camera" visible="false" simulate_depth="false">
+    <origin xyz="0 0 0" rpy="0 0 0" />
+  </xacro:realsense_d435>
   <!-- Force/Torque Sensor -->
   <link name="robot/wrist_3_joint/force_torque_sensor" />

Commit message: Add calibration setup to Gazebo solution config

File: src/ur_gazebo_config/description/ur5e_with_scene_camera_gazebo.xacro (robot description, xacro)
@@ -158,4 +158,11 @@
     </sensor>
   </gazebo>
+  <!-- Dummy link for the checkerboard -->
+  <link name="checkerboard" />
+  <joint name="checkerboard_joint" type="fixed">
+    <parent link="grasp_link" />
+    <child link="checkerboard" />
+    <origin xyz="0.0 0.1 0.0" rpy="0.0 0.0 0.0" />
+  </joint>
   <!-- Gazebo Plugins -->
   <gazebo>
