Commit message: Removed unneeded use_extra_camera xacro arg

File: src/solution_ur_gazebo_config/description/ur5e_gazebo.xacro (robot description, xacro)
@@ -7,5 +7,4 @@
   <xacro:arg name="physical_parameters_file" default="" />
   <xacro:arg name="visual_parameters_file" default="" />
-  <xacro:arg name="use_extra_camera" default="false"/>
   <xacro:arg name="gazebo_renderer" default="ogre"/>
   <!-- Import macros for main hardware components -->
@@ -90,15 +89,13 @@
   </xacro:realsense_d435>
   <!-- Additional Camera -->
-  <xacro:if value="$(arg use_extra_camera)">
-    <link name="extra_scene_camera_link" />
-    <joint name="extra_scene_camera_joint" type="fixed">
-      <parent link="world" />
-      <child link="extra_scene_camera_link" />
-      <origin xyz="-0.3 0.3 0.5" rpy="0.0 0.0 -3.14" />
-    </joint>
-    <xacro:realsense_d435 parent="extra_scene_camera_link" name="extra_camera" visible="false" simulate_depth="false">
-      <origin xyz="0 0 0" rpy="0 0 0" />
-    </xacro:realsense_d435>
-  </xacro:if>
+  <link name="extra_scene_camera_link" />
+  <joint name="extra_scene_camera_joint" type="fixed">
+    <parent link="world" />
+    <child link="extra_scene_camera_link" />
+    <origin xyz="-0.3 0.3 0.5" rpy="0.0 0.0 -3.14" />
+  </joint>
+  <xacro:realsense_d435 parent="extra_scene_camera_link" name="extra_camera" visible="false" simulate_depth="false">
+    <origin xyz="0 0 0" rpy="0 0 0" />
+  </xacro:realsense_d435>
   <!-- Force/Torque Sensor -->
   <link name="robot/wrist_3_joint/force_torque_sensor" />

File: src/ur_gazebo_config/description/ur5e_gazebo.xacro (robot description, xacro)
@@ -7,5 +7,4 @@
   <xacro:arg name="physical_parameters_file" default="" />
   <xacro:arg name="visual_parameters_file" default="" />
-  <xacro:arg name="use_extra_camera" default="false"/>
   <xacro:arg name="gazebo_renderer" default="ogre"/>
   <!-- Import macros for main hardware components -->
