Commit message: Fixes from hardware testing

File: src/ur_hardware_config/description/picknik_007_ur5e.xacro (robot description, xacro)
@@ -91,5 +91,5 @@
     <parent link="base" />
     <child link="environment" />
-    <origin rpy="0 0 0" xyz="0 0 0" />
+    <origin rpy="0 0 0" xyz="0 0 -0.09" />
   </joint>
   <!-- Camera External -->
